File: WTL-Split-Left/WTL-Split-Left.kicad_pcb (KiCad board)
At the start: 2 copper layers, 142.9 x 77.8 mm, 48 parts, among them J1 MJ-4PP-9, U1 ProMicro

Commit message: this project gonna end up in a bin but ok
Connections:
- U1 pad 1: Net-(U1-Pad1) -> col1
- U1 pad 10: Net-(U1-Pad10) -> row1
- U1 pad 11: Net-(U1-Pad11) -> row4
- U1 pad 12: Net-(U1-Pad12) -> row3
- U1 pad 13: Net-(U1-Pad13) -> row2
- U1 pad 14: Net-(U1-Pad14) -> col3
- U1 pad 15: Net-(U1-Pad15) -> col4
- U1 pad 16: Net-(U1-Pad16) -> col5
- U1 pad 17: Net-(U1-Pad17) -> col6
- U1 pad 18: Net-(U1-Pad18) -> col7
- U1 pad 19: Net-(U1-Pad19) -> col8
- U1 pad 20: Net-(U1-Pad20) -> col2
Routing:
- net col8: track 19.0 -> 173.2 mm
- net col7: track 44.0 -> 148.6 mm
- net col6: track 67.0 -> 150.6 mm
- net col5: track 63.1 -> 125.8 mm
- net row1: track 95.2 -> 146.6 mm, vias 0 -> 1
- net row4: track 77.2 -> 121.9 mm, vias 0 -> 1
- net col4: track 63.1 -> 105.0 mm
- net row3: track 95.7 -> 110.2 mm, vias 0 -> 1
- net col1: track 0.00 -> 10.1 mm
- net col3: track 21.0 -> 29.5 mm
- net col2: track 40.1 -> 45.8 mm
- net row2: track 101.4 -> 104.8 mm

Commit message: i'm fucking tired
Parts:
- J1: moved to B.Cu
- moved J1 36.7 mm to (183.4, 23.0), turned to 180 degrees
- moved D5 17.5 mm to (163.5, 27.8)
Routing:
- net GND: track 131.2 -> 183.5 mm, vias 2 -> 0
- net Net-(D7-Pad2): track 20.2 -> 45.6 mm
- net +5V: track 139.8 -> 151.9 mm, vias 2 -> 0
- net Net-(D5-Pad2): track 3.35 -> 14.8 mm
- net row1: track 146.6 -> 153.4 mm
- net row4: track 121.9 -> 127.3 mm, vias 1 -> 0
- net data_r: track 132.6 -> 128.7 mm
- net row3: track 110.2 -> 111.0 mm, vias 1 -> 0
