File: WTL-Split-Right/WTL-Split-Right.kicad_pcb (KiCad board)
At the start: 2 copper layers, 138.1 x 77.8 mm, 46 parts, among them J1 MJ-4PP-9, U1 ProMicro

Commit message: i'm fucking tired
Parts:
- U1: moved to B.Cu
- moved D20 1.77 mm to (174.6, 73.0)
- moved D14 0.79 mm to (177.8, 50.8)
- turned U1 to 90 degrees
Connections:
- U1 pad 10: Net-(U1-Pad10) -> row2
- U1 pad 13: col6 -> Net-(U1-Pad13)
- U1 pad 19: row1 -> row4
- U1 pad 20: col7 -> row3
- U1 pad 7: row2 -> col7
- U1 pad 8: row3 -> col6
- U1 pad 9: row4 -> row1
Routing:
- net col1: track 149.1 -> 181.7 mm
- net row4: track 74.6 -> 102.9 mm, vias 1 -> 0
- net row1: track 149.3 -> 176.9 mm, vias 1 -> 0
- net col5: track 66.8 -> 89.6 mm
- net dara_r: track 152.3 -> 133.4 mm
- net row2: track 127.3 -> 110.6 mm
- net GND: track 141.7 -> 129.7 mm
- net col6: track 50.8 -> 59.2 mm
- net col4: track 105.9 -> 110.5 mm
- net +5V: track 137.0 -> 132.9 mm
- net col7: track 48.3 -> 51.7 mm
- net col2: track 173.5 -> 170.6 mm
- net row3: track 104.1 -> 102.4 mm, vias 1 -> 0
