File: WTL-Split-Right/WTL-Split-Right.kicad_pcb (KiCad board)
At the start: 2 copper layers, 138.1 x 77.8 mm, 46 parts, among them J1 MJ-4PP-9, U1 ProMicro

Commit message: 1.0 version
Parts:
- added REF**: ToolingHole, kicadPepe:ToolingHole, F.Cu at (50.8, 34.9)
- added REF**: ToolingHole, kicadPepe:ToolingHole, F.Cu at (181.0, 38.9)
- added REF**: ToolingHole, kicadPepe:ToolingHole, F.Cu at (65.1, 109.5)
Routing:
- net GND: track 129.7 -> 0.00 mm
- added copper zone on B.Cu, net (none)
- added copper zone on F.Cu, net (none)
- added copper zone on B.Cu, net GND
- added copper zone on F.Cu, net GND
Other:
- board text added: "Willing To Live SplitR"
- board text added: "design by sat1l"

Commit message: I don't remember what i've done
Parts:
- MX21: footprint MX_Only:MXOnly-2U-NoLED -> MX_Only:MXOnly-2U-ReversedStabilizers-NoLED
- moved D1 26.7 mm to (86.5, 38.1), turned to 225 degrees
- moved D7 17.5 mm to (162.7, 38.1)
- moved D22 17.5 mm to (100.8, 95.2)
- moved D20 17.0 mm to (158.0, 76.2)
- moved D13 2.86 mm to (161.1, 49.2), turned to 225 degrees
Routing:
- net GND: track 0.00 -> 129.9 mm
- net row1: track 176.9 -> 136.3 mm
- net Net-(D1-Pad2): track 9.12 -> 26.9 mm
- net Net-(D20-Pad2): track 3.22 -> 14.8 mm
- net Net-(D22-Pad2): track 3.35 -> 14.8 mm
- net Net-(D7-Pad2): track 3.35 -> 14.8 mm
- net +5V: track 132.9 -> 142.9 mm, vias 1 -> 0
- net row2: track 110.6 -> 119.8 mm
- net Net-(D13-Pad2): track 6.35 -> 8.03 mm
- net row4: track 102.9 -> 103.8 mm
- removed copper zone on B.Cu, net (none)
- removed copper zone on F.Cu, net (none)
- removed copper zone on B.Cu, net GND
- removed copper zone on F.Cu, net GND

Commit message: changes shift key on left half from 2u to 2.25u
Other:
- outline, holes or cut-outs redrawn
- net class Default removed
