File: WTL-Split-Plates/WTL-Split-Plates-Left/WTL-Split-Plates-Left.kicad_pcb (KiCad board)
At the start: 2 copper layers, 152.4 x 77.8 mm, 26 parts, among them SW2 KEY_SWITCH

Commit message: I don't remember what i've done
Parts:
- turned REF** to 180 degrees (x2)
