File: WTL-Split-Plates/WTL-Split-Plates-Right/WTL-Split-Plates-Right.kicad_pcb (KiCad board)
At the start: 2 copper layers, 138.1 x 76.2 mm, 23 parts, among them SW2 KEY_SWITCH

Commit message: I don't remember what i've done
Parts:
- turned REF** to 180 degrees
